File: USBToEthernet/USBToEthernet.kicad_pcb (KiCad board)
At the start: 2 copper layers, 0 parts

Commit message: Most placements I think done
Parts:
- added C1: 10uF, Capacitor_SMD:C_0603_1608Metric, F.Cu at (68.4, 96.5)
- added C10: 1uF, Capacitor_SMD:C_0603_1608Metric, F.Cu at (93.1, 111.2)
- added C11: 1uF, Capacitor_SMD:C_0603_1608Metric, F.Cu at (86.5, 106.4)
- added C12: 1uF, Capacitor_SMD:C_0603_1608Metric, F.Cu at (84.4, 104.7)
- added C13: 1uF, Capacitor_SMD:C_0603_1608Metric, F.Cu at (99.8, 107.8)
- added C14: 1uF, Capacitor_SMD:C_0603_1608Metric, F.Cu at (94.1, 97.3)
- added C15: 1uF, Capacitor_SMD:C_0603_1608Metric, F.Cu at (99.8, 104.7)
- added C16: 1uF, Capacitor_SMD:C_0603_1608Metric, F.Cu at (94.7, 111.3)
- added C17: 1uF, Capacitor_SMD:C_0603_1608Metric, F.Cu at (92.5, 97.3)
- added C18: 1uF, Capacitor_SMD:C_0603_1608Metric, F.Cu at (89.9, 111.3)
- added C19: 100nF, Capacitor_SMD:C_0805_2012Metric, F.Cu at (72.3, 100.6)
- added C2: 10uF, Capacitor_SMD:C_0603_1608Metric, F.Cu at (68.5, 93.2)
- added C20: 1uF, Capacitor_SMD:C_0603_1608Metric, F.Cu at (87.2, 110.2)
- added C21: 1uF, Capacitor_SMD:C_0603_1608Metric, F.Cu at (91.5, 111.2)
- added C22: 1uF, Capacitor_SMD:C_0603_1608Metric, F.Cu at (99.9, 103.0)
- added C23: 1uF, Capacitor_SMD:C_0603_1608Metric, F.Cu at (96.3, 111.8)
- added C24: 1uF, Capacitor_SMD:C_0603_1608Metric, F.Cu at (84.4, 103.1)
- added C25: 1uF, Capacitor_SMD:C_0603_1608Metric, F.Cu at (89.6, 98.5)
- added C26: 24pF, Capacitor_SMD:C_0603_1608Metric, F.Cu at (81.2, 98.6)
- added C27: 24pF, Capacitor_SMD:C_0603_1608Metric, F.Cu at (84.5, 95.7)
- added C3: 10uF, Capacitor_SMD:C_0603_1608Metric, F.Cu at (64.8, 114.3)
- added C4: 10uF, Capacitor_SMD:C_0603_1608Metric, F.Cu at (72.0, 107.5)
- added C5: 0.022uF, Capacitor_SMD:C_0603_1608Metric, F.Cu at (112.6, 112.7)
- added C6: 0.022uF, Capacitor_SMD:C_0603_1608Metric, F.Cu at (117.7, 117.0)
- added C7: 0.022uF, Capacitor_SMD:C_0603_1608Metric, F.Cu at (117.6, 93.7)
- added C8: 0.022uF, Capacitor_SMD:C_0603_1608Metric, F.Cu at (113.1, 97.7)
- added C9: 100nF, Capacitor_SMD:C_0603_1608Metric, F.Cu at (86.8, 116.2)
- added FB1: 120@100, Inductor_SMD:L_0603_1608Metric, F.Cu at (92.2, 94.0)
- added FB2: 120@100, Inductor_SMD:L_0603_1608Metric, F.Cu at (92.7, 113.7)
- added FB3: 120@100, Inductor_SMD:L_0603_1608Metric, F.Cu at (87.2, 112.0)
- added FB4: 120@100, Inductor_SMD:L_0603_1608Metric, F.Cu at (105.2, 86.4)
- added FB5: 120@100, Inductor_SMD:L_0603_1608Metric, F.Cu at (89.6, 95.3)
- added J1: USB_A, USB_AP_S_RA_SMT:CONN_USB-AP-S-RA-SMT_ADM, F.Cu at (54.4, 103.8)
- added J2: L836-1J1T-43, L836-1J1T-43:BEL_L836-1J1T-43, F.Cu at (125.0, 105.5)
- added R1: 12k, Resistor_SMD:R_0603_1608Metric, F.Cu at (88.9, 113.7)
- added R10: 49.9, Resistor_SMD:R_0603_1608Metric, F.Cu at (110.4, 76.5)
- added R11: 49.9, Resistor_SMD:R_0603_1608Metric, F.Cu at (117.2, 74.0)
- added R12: 49.9, Resistor_SMD:R_0603_1608Metric, F.Cu at (117.4, 77.2)
- added R13: 10k, Resistor_SMD:R_0603_1608Metric, F.Cu at (84.0, 117.0)
- added R2: 8.06k, Resistor_SMD:R_0603_1608Metric, F.Cu at (99.9, 101.2)
- added R3: 1k, Resistor_SMD:R_0603_1608Metric, F.Cu at (131.1, 94.0)
- added R4: 1k, Resistor_SMD:R_0603_1608Metric, F.Cu at (128.2, 118.1)
- added R5: 49.9, Resistor_SMD:R_0603_1608Metric, F.Cu at (98.0, 77.4)
- added R6: 49.9, Resistor_SMD:R_0603_1608Metric, F.Cu at (97.7, 80.5)
- added R7: 49.9, Resistor_SMD:R_0603_1608Metric, F.Cu at (104.4, 73.6)
- added R8: 49.9, Resistor_SMD:R_0603_1608Metric, F.Cu at (104.4, 76.6)
- added R9: 49.9, Resistor_SMD:R_0603_1608Metric, F.Cu at (110.2, 73.6)
- added SW1: SW_Push, Button_Switch_SMD:SW_SPST_PTS645Sx43SMTR92, F.Cu at (80.2, 112.5)
- added U1: LAN7500-ABJZ, Package_DFN_QFN:QFN-56-1EP_8x8mm_P0.5mm_EP5.9x5.9mm, F.Cu at (93.5, 104.8)
- added U2: NCP1117-3.3_SOT223, Package_TO_SOT_SMD:SOT-223-3_TabPin2, F.Cu at (74.0, 95.0)
- added U3: 93LCxxAxxOT, Package_TO_SOT_SMD:SOT-23-6, F.Cu at (99.5, 115.0)
- added U4: USBLC6-2SC6, Package_TO_SOT_SMD:SOT-23-6, F.Cu at (72.4, 103.8)
- added U6: AMS1117-1.2, Package_TO_SOT_SMD:SOT-223-3_TabPin2, F.Cu at (70.2, 112.2)
- added Y1: 25Mhz, Crystal:Crystal_SMD_SeikoEpson_FA238V-4Pin_3.2x2.5mm, F.Cu at (84.3, 98.5)
Routing:
- net /TR0: track 0.00 -> 19.7 mm
- net +3V3: track 0.00 -> 0.54 mm
- net GND: vias 0 -> 1
Other:
- board outline added: 81.4 x 37.3 mm

Commit message: Fried ahh PCB layout and routing
Parts:
- C14, C17, C25, FB1, FB5, R1: moved to B.Cu
- C19: footprint Capacitor_SMD:C_0805_2012Metric -> Capacitor_SMD:C_0603_1608Metric
- J1: value USB_A -> 0480372200; footprint USB_AP_S_RA_SMT:CONN_USB-AP-S-RA-SMT_ADM -> USB_A_Plug:MOLEX_0480372200
- moved R11 37.0 mm to (88.4, 97.3), turned to -90 degrees
- moved R12 33.9 mm to (90.1, 97.3), turned to -90 degrees
- moved R9 30.1 mm to (91.8, 97.4), turned to -90 degrees
- moved R10 26.9 mm to (93.3, 97.4), turned to -90 degrees
- moved R7 25.3 mm to (95.2, 97.2), turned to -90 degrees
- moved R8 21.9 mm to (96.9, 97.2), turned to -90 degrees
- moved R5 20.7 mm to (100.0, 98.0), turned to 180 degrees
- moved R6 19.2 mm to (99.9, 99.6), turned to 180 degrees
- moved FB4 10.4 mm to (98.1, 94.0), turned to -90 degrees
- moved J1 7.09 mm to (61.5, 103.9)
- moved R3 5.64 mm to (125.5, 93.3)
- moved C8 5.58 mm to (107.6, 97.1)
- moved C6 5.33 mm to (112.4, 116.4)
- moved C5 5.33 mm to (107.3, 112.1)
- moved J2 5.33 mm to (119.7, 104.9)
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Connections:
- J1 pad 2: /D- -> /D+
- J1 pad 3: /D+ -> /D-
Routing:
- net +3V3: track 0.54 -> 170.7 mm, vias 0 -> 11
- net +1V2: track 0.49 -> 120.8 mm, vias 0 -> 7
- net /LED0: track 0.00 -> 50.1 mm, vias 0 -> 1
- net /LED1: track 0.00 -> 40.8 mm, vias 0 -> 1
- net /LED2: track 0.00 -> 39.5 mm, vias 0 -> 2
- net /RESET: track 0.00 -> 37.6 mm, vias 0 -> 2
- net /VBUS: track 0.43 -> 28.8 mm
- net /VDD12A: track 0.25 -> 26.9 mm, vias 0 -> 6
- net /DOut+: track 0.00 -> 18.5 mm
- net /DOut-: track 0.00 -> 18.5 mm
- net /TR0: track 19.7 -> 36.4 mm
- net /XO: track 0.00 -> 12.1 mm
- net /XI: track 0.10 -> 11.0 mm
- net /VDD12PLL: track 0.14 -> 7.92 mm, vias 0 -> 1
- net /MISO: track 0.00 -> 7.20 mm, vias 0 -> 2
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Other:
- board size 81.4 x 37.3 mm -> 5.1 x 17.6 mm

Commit message: Revamped the PCB
Parts:
- C14, R1: moved to F.Cu
- C16, C22, C23, C24, FB2, FB3: moved to B.Cu
- moved R1 34.8 mm to (83.7, 79.8), turned to -90 degrees
- moved C10 32.3 mm to (85.5, 79.9), turned to 90 degrees
- moved FB2 30.3 mm to (81.3, 85.4), turned to 0 degrees
- moved U3 29.4 mm to (79.3, 90.9)
- moved C23 29.1 mm to (81.4, 87.0), turned to 180 degrees
- moved FB3 28.6 mm to (81.8, 83.9)
- moved C18 28.5 mm to (81.3, 84.9), turned to 180 degrees
- moved C20 27.3 mm to (82.1, 83.4)
- moved C11 26.1 mm to (87.2, 80.3), turned to 90 degrees
- moved C15 24.8 mm to (81.4, 88.1), turned to 180 degrees
- moved C24 23.2 mm to (88.8, 80.3), turned to 90 degrees
- moved C22 23.1 mm to (81.9, 88.5), turned to 180 degrees
- moved C16 22.8 mm to (95.7, 88.4), turned to 0 degrees
- moved C26 22.1 mm to (88.8, 78.6)
- moved Y1 21.9 mm to (91.9, 78.5)
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Connections:
- U1 pad 43: /TR0- -> /TR0+
- U1 pad 44: /TR0+ -> /TR0-
- U1 pad 51: /TR2- -> /TR2+
- U1 pad 52: /TR2+ -> /TR2-
Routing:
- net GND: track 0.00 -> 83.6 mm, vias 0 -> 42
- net /TR0: track 36.4 -> 72.0 mm, vias 0 -> 6
- net /RESET: track 37.6 -> 22.3 mm
- net +1V2: track 120.8 -> 134.6 mm, vias 7 -> 6
- net /TR2+: track 2.91 -> 15.0 mm
- net /TR2-: track 2.91 -> 14.8 mm
- net /TR1+: track 3.03 -> 13.5 mm
- net /TR1-: track 3.53 -> 13.8 mm
- net /TR3-: track 3.27 -> 12.3 mm
- net /TR3+: track 3.81 -> 12.3 mm
- net /TR0-: track 3.86 -> 11.0 mm
- net /TR0+: track 4.45 -> 11.0 mm
- net +3V3: track 170.7 -> 176.4 mm, vias 11 -> 13
- net /XO: track 12.1 -> 6.55 mm
- net Net-(J2-Pad14): track 0.00 -> 4.53 mm
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- added copper zone on B.Cu, net GND
- added copper zone on F.Cu, net GND
Other:
- board size 5.1 x 17.6 mm -> 61.3 x 30 mm
- board text added: "Dynix"
